File: pcb/TensiometroDigital/nxp_lpc1769_chip.sch (KiCad schematic (older format))
At the start: 30 parts

Commit message: Finalizado: SCH, PCB, GABINETE, DRAWINGS. FALTA: GERBERS, BOM e Informe
Parts:
- removed SW?: SW_SPST, symbol SW_SPST
- added C12, C13: 5pF, Capacitors_SMD:C_0805_HandSoldering, symbol C
- added D1, D2: LED, LEDs:LED_0402, symbol LED
- added D7: 1N4448WS-7-F, Diodes_SMD:D_SOD-323, symbol D
- added JP1: Jumper, Socket_Strips:Socket_Strip_Straight_1x02_Pitch2.54mm, symbol Jumper
- added R13, R16: 1k5, Resistors_SMD:R_0805_HandSoldering, symbol R
- added R22: 100K, Resistors_SMD:R_0805_HandSoldering, symbol R
- added RTC_BAT1: CR2032, footprints:CR2032_VERTICAL_HOLDER_S8401-46, symbol Battery_Cell
- added TP10: SSEL0, footprints:TestPoint_THTPad_D1.5mm_Drill0.7mm, symbol TEST
- added TP11: DATA, footprints:TestPoint_THTPad_D1.5mm_Drill0.7mm, symbol TEST
- added TP12: MOSI0, footprints:TestPoint_THTPad_D1.5mm_Drill0.7mm, symbol TEST
- added TP13: RTCK, footprints:TestPoint_THTPad_D1.5mm_Drill0.7mm, symbol TEST
- added TP14: SENS, footprints:TestPoint_THTPad_D1.5mm_Drill0.7mm, symbol TEST
- added TP15: FLTR, footprints:TestPoint_THTPad_D1.5mm_Drill0.7mm, symbol TEST
- added TP16: RSTOUT, footprints:TestPoint_THTPad_D1.5mm_Drill0.7mm, symbol TEST
- added TP3: START, footprints:TestPoint_THTPad_D1.5mm_Drill0.7mm, symbol TEST
- added TP4: SEL, footprints:TestPoint_THTPad_D1.5mm_Drill0.7mm, symbol TEST
- added TP5: SSEL1, footprints:TestPoint_THTPad_D1.5mm_Drill0.7mm, symbol TEST
- added TP6: SCK1, footprints:TestPoint_THTPad_D1.5mm_Drill0.7mm, symbol TEST
- added TP7: MISO1, footprints:TestPoint_THTPad_D1.5mm_Drill0.7mm, symbol TEST
- added TP8: MOSI1, footprints:TestPoint_THTPad_D1.5mm_Drill0.7mm, symbol TEST
- added TP9: SCK0, footprints:TestPoint_THTPad_D1.5mm_Drill0.7mm, symbol TEST
- added Y2: 32.768KHz, footprints:Crystal_SMD_2012-2pin_2.0x1.2mm_HandSoldering, symbol Crystal
- C10, C11: renamed from C?; footprint (none) -> Capacitors_SMD:C_0805_HandSoldering; manf# (none) -> CBR08C180FAGAC
- C14, C15, C16, C17: renamed from C?; footprint (none) -> Capacitors_SMD:C_0805_HandSoldering; manf# (none) -> C0805C103JARACTU
- C18, C19, C20, C21, C22, C23: renamed from C?; footprint (none) -> Capacitors_SMD:C_0805_HandSoldering; manf# (none) -> C0805X104J5RACAUTO
- D5: renamed from D?; footprint (none) -> Diodes_SMD:D_SOD-323; manf# (none) -> PMEG1020EA,115
- D6: renamed from D?; value 4448 -> 1N4448WS-7-F; footprint (none) -> Diodes_SMD:D_SOD-323; manf# (none) -> 1N4448WS-7-F
- J3: renamed from J?; value Conn_01x08 -> Programacion; footprint (none) -> Socket_Strips:Socket_Strip_Straight_1x08_Pitch2.54mm
- JP2: renamed from JP?; footprint (none) -> Socket_Strips:Socket_Strip_Straight_1x02_Pitch2.54mm
- L2: renamed from L?; value Ferrite_Bead -> BK1608HS220-T; footprint (none) -> Inductors_SMD:L_0603_HandSoldering; Field4 https://www.digikey.com/product-detail/es/taiyo-yuden/BK160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 -> (none); manf# (none) -> BK1608HS220-T
- R21: renamed from R?; footprint (none) -> Resistors_SMD:R_0805_HandSoldering; manf# (none) -> SG73G2ATTD1002D
- R23: renamed from R?; footprint (none) -> Resistors_SMD:R_0805_HandSoldering; manf# (none) -> RT0805DRD0712KL
- R24, R25, R26, R27, R28: renamed from R?; footprint (none) -> Resistors_SMD:R_0805_HandSoldering; manf# (none) -> AC0805FR-070RL
- R29, R30: renamed from R?; footprint (none) -> Resistors_SMD:R_0805_HandSoldering; manf# (none) -> SG73G2ATTD3301D
- U8: renamed from U?; footprint Package_QFP:LQFP-100_14x14mm_P0.5mm -> footprints:LQFP-100_14x14mm_P0.5mm; symbol LPC1769FBD100 -> LPC1769FBD100-RESCUE-TensiometroDigital-RESCUE-TensiometroDigital; manf# (none) -> LPC1769FBD100,551
- U9: renamed from U?; manf# (none) -> 24LC64-I/SN
- Y1: renamed from Y?; footprint (none) -> footprints:Crystal_SMD_Abracon_ABM3C-4pin_5.0x3.2mm; manf# (none) -> ABM3B-12.000MHZ-B2-T
Connections:
- net TCK_SWDCLK is gone; now on net TCLK_SWDCLK: U8.5 (TCK/SWDCLK)
- net +3V3: now also JP1.1
- net DATA: now also TP11.1
- net GND: now also C12.2, C13.2, D2.1 (K), RTC_BAT1.2 (-)
- net LED_BUZZER: now also U8.35 (P1[21]); no longer U8.44 (P1[28])
- net MISO1: now also TP7.1
- net MOSI0: now also TP12.1
- net MOSI1: now also TP8.1
- net P0[19]: no longer R29.2, U9.5 (SDA)
- net P0[20]: no longer R30.2, U9.6 (SCL)
- net SCK0: now also TP9.1
- net SCK1: now also TP6.1
- net SSEL0: now also TP10.1
- net SSEL1: now also TP5.1
- net VBAT: now also U8.19 (VBAT), D7.1 (K); no longer U8.10 (VDDA)
- net VDD_3V3: now also R13.1
- net VREF: now also U8.10 (VDDA); no longer U8.19 (VBAT)
- net RTCK: now reaches U8.100 (RTCK)
- net RTCK: now also TP13.1
- net ~RSTOUT: now reaches U8.14 (~RSTOUT~)
- net ~RSTOUT: now also D1.1 (K), TP16.1
- net at U8.16 (RTCX1): now also C12.1, Y2.1
- net at U8.18 (RTCX2): now also R22.1
- net BOMBA: now reaches U8.32 (P1[18])
- net VALVULA: now reaches U8.34 (P1[20])
- net ~START: now reaches U8.50 (P2[13])
- net ~START: now also TP3.1
- net ~SELECT: now reaches U8.51 (P2[12])
- net ~SELECT: now also TP4.1
- net STATUS_LED: now reaches U8.56 (P0[22])
- net STATUS_LED: now also R16.1
- net SCL_EEPROM: now reaches U8.58 (P0[20])
- net SCL_EEPROM: now also R30.2, U9.6 (SCL)
- net SDA_EEPROM: now reaches U8.59 (P0[19])
- net SDA_EEPROM: now also R29.2, U9.5 (SDA)
- net SENSOR: now reaches U8.8 (P0[24])
- net SENSOR: now also TP14.1
- net ~ARESET: now reaches U8.86 (P1[17])
- net FILTER: now reaches U8.9 (P0[23])
- net FILTER: now also TP15.1
- net at D5.2 (A): now also JP1.2
- net ~RESET renamed ~MRESET
- new net: D7.2 (A), RTC_BAT1.1 (+)
- new net: C13.1, R22.2, Y2.2
- new net: D1.2 (A), R13.2
- new net: D2.2 (A), R16.2
- no-connect marks 1 -> 52
Other:
- note added: "ALIMENTACIÓN LPC1769\n"
- note added: "JP1 abierto cuando se programa."
- note added: "JP2 normalmente en cortocircuito. \nPuede ser utilizado paramediciones de\nconsumo de corriente del micro."
- note added: "LED DE ESTADO"
- note added: "RESET LED"
- note added: "Reset Display"
- note added: "TEST POINTS"
- note removed: "- Reset Display"
- note removed: "ALIMENTACIÓN\n"
- note removed: "Colocar XTAL RTC?? Viene al caso?"
- note removed: "JP normalmente en cortocircuito. \nPuede ser utilizado paramediciones de\nconsumo de corriente del micro."
- note removed: "SW abierto cuando se programa."
- moved on the sheet: C10, C11, C14, C15, C16, C17, C18, C19, C20, C21, C22, C23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
