File: pcb/TensiometroDigital/TensiometroDigital.kicad_pcb (KiCad board)
At the start: 2 copper layers, 100 x 100 mm, 131 parts, among them J1 SD_Card, J2 BAT 9V, J3 Programacion, J4 VALVE, J5 AIR PUMP, M3 MountingHole_3.2mm_M3, Q1 BC557, Q2 TIP31, Q3 TIP31, SW2 SW_SPDT, SW3 SW_DPST, SW4 SW_DPST, SW5 SW_DPST, U1 LM358, U10 MPXV5050GP, U11 BAV199, U2 4N25, U3 display_nokia5110, U4 LM8364BALMF20/NOPBTR-ND, U5 BAV199, U6 LM2575-3.3, U7 LM2940-5V, U8 LPC1769FBD100, U9 24LC64, Y1 12MHz, Y2 32.768KHz

Commit message: TP FINALIZADO. FALTA CREAR EL ZIP
Other:
- board text added: "- SD"
- board text added: "Display LCD 5110"
- board text added: "GND"
- board text added: "LPC1769"
Changed lines of the file:
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@@
     (area 99.924999 49.924999 200.075001 150.075001)
     (thickness 1.6)
-    (drawings 173)
+    (drawings 178)
     (tracks 1550)
     (zones 0)
@@
     (tags "sd card")
     (attr smd)
-    (fp_text reference J1 (at 13.24348 -7.21738 360) (layer F.SilkS)
+    (fp_text reference J1 (at 15.57188 1.32842 450) (layer F.SilkS)
       (effects (font (size 1 1) (thickness 0.25)))
     )
@@
       (xy 0.164043 -2.914165)) (layer F.SilkS) (width 0.01))
   )
+  (gr_text LPC1769 (at 150 111) (layer F.SilkS)
+    (effects (font (size 1 1) (thickness 0.25)))
+  )
+  (gr_text GND (at 172 63 90) (layer F.SilkS)
+    (effects (font (size 1 1) (thickness 0.25)))
+  )
+  (gr_text RST (at 154 64 90) (layer F.SilkS)
+    (effects (font (size 1 1) (thickness 0.25)))
+  )
+  (gr_text "Display LCD 5110" (at 163 62.5) (layer F.SilkS)
+    (effects (font (size 1 1) (thickness 0.25)))
+  )
+  (gr_text "- SD" (at 109 62 90) (layer F.SilkS)
+    (effects (font (size 1 1) (thickness 0.25)))
+  )
   (gr_text "Tensiómetro Digital" (at 150 35) (layer Cmts.User)
